Commit message: Fix CollisionChecker build and GJK warm-start false-negatives
- Include pinocchio/collision/{collision,distance}.hpp so the
  computeCollisions/computeDistances overloads are visible.
- Pin GeometryObject constructor calls to the non-deprecated
  (parent_joint, parent_frame, SE3, geometry) order; the old
  (parent_frame, parent_joint, geometry, SE3) signature is gone in
  Pinocchio 3.x and was failing template resolution.
- Include coal/BVH/BVH_model.h on the mesh path so BVHModelBase's
  inheritance from CollisionGeometry is visible to the implicit
  shared_ptr conversion.
- Disable coal's deprecated cached_gjk_guess warm-start on every
  CollisionRequest/DistanceRequest after rebuild. Pinocchio enables it
  by default (geometry.hxx) and it produces false-negatives when a
  colliding query follows a sequence of non-colliding queries on the
  same pair, because GJK warm-starts from a stale separating direction.
- check_path: take the row-major PathMatrix by value so numpy's C-order
  (N, nq) arrays are interpreted correctly. The default MatrixXd is
  column-major and was silently transposing the path.
- Lengthen L2's collision box in tests/collision_two_link.urdf so a
  folded q=[0, pi] produces a base<->L2 (non-adjacent) collision. The
  prior geometry only collided L1<->L2, which the default policy
  disables.
- Fix tests/test_collision.py to compute COLLISION_URDF_PATH locally
  instead of relative-importing from conftest (tests/ isn't a package).

https://claude.ai/code/session_01TiEkni9M9ZJC88LmvJwUyf

File: tests/collision_two_link.urdf (robot description, URDF)
Before this commit: robot collision_two_link, 3 links, 2 joints
Links:
- link L2: geometry collision box size=0.05 0.05 0.50
